Commit message: Added bullet interface.

File: models/yumi/yumi.urdf (robot description, URDF)
Before this commit: robot yumi, 22 links, 21 joints
Links:
- link gripper_l_base: geometry collision mesh filename=meshes/gripper/coarse/base.stl; visual mesh filename=meshes/gripper/base.stl
- link gripper_l_finger_l: geometry collision mesh filename=meshes/gripper/coarse/finger.stl; visual mesh filename=meshes/gripper/finger.stl
- link gripper_l_finger_r: geometry collision mesh filename=meshes/gripper/coarse/finger.stl; visual mesh filename=meshes/gripper/finger.stl
- link gripper_r_base: geometry collision mesh filename=meshes/gripper/coarse/base.stl; visual mesh filename=meshes/gripper/base.stl
- link gripper_r_finger_l: geometry collision mesh filename=meshes/gripper/coarse/finger.stl; visual mesh filename=meshes/gripper/finger.stl
- link gripper_r_finger_r: geometry collision mesh filename=meshes/gripper/coarse/finger.stl; visual mesh filename=meshes/gripper/finger.stl
- link yumi_body: geometry collision mesh filename=meshes/coarse/body.stl; visual mesh filename=meshes/body.stl
- link yumi_link_1_l: geometry collision mesh filename=meshes/coarse/link_1.stl; visual mesh filename=meshes/link_1.stl
- link yumi_link_1_r: geometry collision mesh filename=meshes/coarse/link_1.stl; visual mesh filename=meshes/link_1.stl
- link yumi_link_2_l: geometry collision mesh filename=meshes/coarse/link_2.stl; visual mesh filename=meshes/link_2.stl
- link yumi_link_2_r: geometry collision mesh filename=meshes/coarse/link_2.stl; visual mesh filename=meshes/link_2.stl
- link yumi_link_3_l: geometry collision mesh filename=meshes/coarse/link_3.stl; visual mesh filename=meshes/link_3.stl
- link yumi_link_3_r: geometry collision mesh filename=meshes/coarse/link_3.stl; visual mesh filename=meshes/link_3.stl
- link yumi_link_4_l: geometry collision mesh filename=meshes/coarse/link_4.stl; visual mesh filename=meshes/link_4.stl
- link yumi_link_4_r: geometry collision mesh filename=meshes/coarse/link_4.stl; visual mesh filename=meshes/link_4.stl
- link yumi_link_5_l: geometry collision mesh filename=meshes/coarse/link_5.stl; visual mesh filename=meshes/link_5.stl
- link yumi_link_5_r: geometry collision mesh filename=meshes/coarse/link_5.stl; visual mesh filename=meshes/link_5.stl
- link yumi_link_6_l: geometry collision mesh filename=meshes/coarse/link_6.stl; visual mesh filename=meshes/link_6.stl
- link yumi_link_6_r: geometry collision mesh filename=meshes/coarse/link_6.stl; visual mesh filename=meshes/link_6.stl
- link yumi_link_7_l: geometry collision mesh filename=meshes/coarse/link_7.stl; visual mesh filename=meshes/link_7.stl
- link yumi_link_7_r: geometry collision mesh filename=meshes/coarse/link_7.stl; visual mesh filename=meshes/link_7.stl
